Commit message: update

File: robotiq/robotiq_s_model_visualization/cfg/robotiq_hand_macro.urdf.xacro (robot description, xacro)
@@ -632,5 +632,5 @@
     </gazebo>
   </xacro:macro>
-  <xacro:macro name="robotiq_hand" params="prefix *origin reflect parent">
+  <xacro:macro name="robotiq_hand" params="prefix *origin parent">
     <!-- joint attaching parent link to robotiq hand -->
     <joint name="${prefix}robotiq_hand_joint" type="fixed">

Commit message: update

File: robotiq/robotiq_s_model_visualization/cfg/robotiq_hand_macro.urdf.xacro (robot description, xacro)
@@ -711,4 +711,11 @@
       <limit lower="0" upper="0" effort="60" velocity="-1"/>
     </joint>
+    <!-- Grasping frame -->
+    <link name="grasping_frame"/>
+    <joint name="grasping_frame_joint" type="fixed">
+      <parent link="${prefix}palm"/>
+      <child link="grasping_frame"/>
+      <origin xyz="0 0 1.57" rpy="0.0455 0.0214 0"/>
+    </joint>
     <gazebo reference="${prefix}palm_finger_middle_joint">
       <implicitSpringDamper>1</implicitSpringDamper>

Commit message: update

File: robotiq/robotiq_s_model_visualization/cfg/robotiq_hand_macro.urdf.xacro (robot description, xacro)
@@ -716,5 +716,5 @@
       <parent link="${prefix}palm"/>
       <child link="grasping_frame"/>
-      <origin xyz="0 0 1.57" rpy="0.0455 0.0214 0"/>
+      <origin xyz="0 0.1 0.01" rpy="0 -1.5708 3.14159"/>
     </joint>
     <gazebo reference="${prefix}palm_finger_middle_joint">

Commit message: update

File: robotiq/robotiq_s_model_visualization/cfg/robotiq_hand_macro.urdf.xacro (robot description, xacro)
@@ -7,4 +7,8 @@
 -->
 <robot xmlns:xacro="http://www.ros.org/wiki/xacro" name="robotiq_hand">
+        <!-- Constants -->
+  <xacro:property name="M_PI" value="3.14159"/>
+    <!-- Gripper frame -->
+  <xacro:property name="grasp_frame_radius" value="0.001" />
   <xacro:macro name="robotiq_finger" params="prefix">
     <!-- Link list -->
@@ -21,5 +25,5 @@
       </visual>
       <collision>
-        <origin rpy="0 0 0" xyz="0 0 0"/>
+        <origin xyz="0 0 0" rpy="0 0 0" />
         <geometry>
           <mesh filename="package://robotiq_s_model_visualization/meshes/s-model_articulated/collision/link_0.STL" />
@@ -42,5 +46,5 @@
     <link name="${prefix}link_1">
       <visual>
-        <origin rpy="0 0 ${3.1416/2}" xyz="0 0.05717 0"/>
+        <origin xyz="0 0.05717 0" rpy="0 0 ${M_PI/2}" />
         <geometry>
           <mesh filename="package://robotiq_s_model_visualization/meshes/s-model_articulated/visual/link_1.STL" />
@@ -49,5 +53,5 @@
       </visual>
       <collision>
-        <origin rpy="0 0 ${3.1416/2}" xyz="0 0.05717 0"/>
+        <origin xyz="0 0.05717 0" rpy="0 0 ${M_PI/2}" />
         <geometry>
           <mesh filename="package://robotiq_s_model_visualization/meshes/s-model_articulated/collision/link_1.STL"/>
@@ -58,5 +62,5 @@
       </collision>
       <inertial>
-        <origin rpy="0 0 ${3.1416/2}" xyz="0.00053 0.03218 0"/>
+        <origin xyz="0.00053 0.03218 0" rpy="0 0 ${M_PI/2}" />
         <mass value="0.047"/>
         <inertia ixx= "0.00000499332"
@@ -75,5 +79,5 @@
     <link name="${prefix}link_2">
       <visual>
-        <origin rpy="0 0 ${3.1416/2}" xyz="0 0.03810 0.0075"/>
+        <origin xyz="0 0.03810 0.0075" rpy="0 0 ${M_PI/2}" />
         <geometry>
           <mesh filename="package://robotiq_s_model_visualization/meshes/s-model_articulated/visual/link_2.STL" />
@@ -82,5 +86,5 @@
       </visual>
       <collision>
-        <origin rpy="0 0 ${3.1416/2}" xyz="0 0.03810 0.0075"/>
+        <origin xyz="0 0.03810 0.0075" rpy="0 0 ${M_PI/2}" />
           <geometry>
             <mesh filename="package://robotiq_s_model_visualization/meshes/s-model_articulated/collision/link_2.STL"/>
@@ -89,5 +93,5 @@
       </collision>
       <inertial>
-        <origin rpy="0 0 ${3.1416/2}" xyz="0.00048 0.02167 0.00018"/>
+        <origin xyz="0.00048 0.02167 0.00018" rpy="0 0 ${M_PI/2}" />
         <mass value="0.03284"/>
         <inertia ixx="0.00000348008"
@@ -120,5 +124,5 @@
       </collision>
       <inertial>
-        <origin rpy="0 0 0" xyz="0.01626 0.00049 0.0002"/>
+        <origin xyz="0.01626 0.00049 0.0002" rpy="0 0 0" />
         <mass value="0.03354"/>
         <inertia ixx="0.00000305151"
@@ -137,5 +141,5 @@
     <link name="${prefix}link_proximal_actuating_hinge">
       <visual>
-        <origin rpy="0 0 0" xyz="0.01429 0 0"/>
+        <origin xyz="0.01429 0 0" rpy="0 0 0" />
         <geometry>
           <box size="0.02858 .0075 .002"/>
@@ -143,5 +147,5 @@
       </visual>
       <collision>
-        <origin rpy="0 0 0" xyz="0.01429 0 0"/>
+        <origin xyz="0.01429 0 0" rpy="0 0 0" />
          <geometry>
           <box size="0.02858 .0075 .002"/>
@@ -149,5 +153,5 @@
       </collision>
       <inertial>
-        <origin rpy="0 0 0" xyz="0.0012 -0.00162 -0.00161"/>
+        <origin xyz="0.0012 -0.00162 -0.00161" rpy="0 0 0" />
         <mass value="0.02647"/>
         <inertia ixx= "0.00000156447"
@@ -166,5 +170,5 @@
     <link name="${prefix}link_paraproximal_actuating_hinge">
       <visual>
-        <origin rpy="0 0 0" xyz="0.01143 0 0"/>
+        <origin xyz="0.01143 0 0" rpy="0 0 0" />
         <geometry>
           <box size="0.02286 .0075 .002"/>
@@ -172,5 +176,5 @@
       </visual>
       <collision>
-        <origin rpy="0 0 0" xyz="0.01143 0 0"/>
+        <origin xyz="0.01143 0 0" rpy="0 0 0" />
          <geometry>
           <box size="0.02286 .0075 .002"/>
@@ -178,5 +182,5 @@
       </collision>
       <inertial>
-        <origin rpy="0 0 0" xyz="0.0064 0 0"/>
+        <origin xyz="0.0064 0 0" rpy="0 0 0" />
         <!-- copied from proximal_actuating_hinge -->
         <mass value="0.00362"/>
@@ -196,5 +200,5 @@
     <link name="${prefix}link_proximal_actuating_bar">
       <visual>
-        <origin rpy="0 0 0" xyz="0.026789 0 0"/>
+        <origin xyz="0.026789 0 0" rpy="0 0 0" />
         <geometry>
           <box size="0.05398 .0075 .002"/>
@@ -202,5 +206,5 @@
       </visual>
       <collision>
-        <origin rpy="0 0 0" xyz="0.026789 0 0"/>
+        <origin xyz="0.026789 0 0" rpy="0 0 0" />
          <geometry>
           <box size="0.05398 .0075 .002"/>
@@ -208,5 +212,5 @@
       </collision>
       <inertial>
-        <origin rpy="0 0 0" xyz="0.02699 -0.00122 0"/>
+        <origin xyz="0.02699 -0.00122 0" rpy="0 0 0" />
         <mass value="0.00659"/>
         <inertia ixx= "0.00000008348"
@@ -225,5 +229,5 @@
     <link name="${prefix}link_paraproximal_bar">
       <visual>
-        <origin rpy="0 0 0" xyz="0.02885 0 0"/>
+        <origin xyz="0.02885 0 0" rpy="0 0 0" />
         <geometry>
           <box size="0.05770 .0075 .002"/>
@@ -231,5 +235,5 @@
       </visual>
       <collision>
-        <origin rpy="0 0 0" xyz="0.02885 0 0"/>
+        <origin xyz="0.02885 0 0" rpy="0 0 0" />
          <geometry>
           <box size="0.05770 .0075 .002"/>
@@ -237,5 +241,5 @@
       </collision>
       <inertial>
-        <origin rpy="0 0 0" xyz="0.02858 -0.00129 0"/>
+        <origin xyz="0.02858 -0.00129 0" rpy="0 0 0" />
         <mass value="0.00732"/>
         <inertia ixx= "0.00000009065"
@@ -254,5 +258,5 @@
     <link name="${prefix}link_median_actuating_hinge">
       <visual>
-        <origin rpy="0 0 0" xyz="0 0 0"/>
+        <origin xyz="0 0 0" rpy="0 0 0" />
         <geometry>
           <box size=".02 .02 .002"/>
@@ -260,5 +264,5 @@
       </visual>
       <collision>
-        <origin rpy="0 0 0" xyz="0 0 0"/>
+        <origin xyz="0 0 0" rpy="0 0 0" />
          <geometry>
           <box size=".02 .02 .002"/>
@@ -266,5 +270,5 @@
       </collision>
       <inertial>
-        <origin rpy="0 0 0" xyz="0.0092 0.00514 0"/>
+        <origin xyz="0.0092 0.00514 0" rpy="0 0 0" />
         <mass value="0.00359"/>
         <inertia ixx= "0.00000024735"
@@ -283,5 +287,5 @@
     <link name="${prefix}link_median_bar">
       <visual>
-        <origin rpy="0 0 0" xyz="0.01905 0 0"/>
+        <origin xyz="0.01905 0 0" rpy="0 0 0" />
         <geometry>
           <box size="0.0381 .0075 .002"/>
@@ -289,5 +293,5 @@
       </visual>
       <collision>
-        <origin rpy="0 0 0" xyz="0.01905 0 0"/>
+        <origin xyz="0.01905 0 0" rpy="0 0 0" />
          <geometry>
           <box size="0.0381 .0075 .002"/>
@@ -295,5 +299,5 @@
       </collision>
       <inertial>
-        <origin rpy="0 0 0" xyz="0.01905 -0.00107 0"/>
+        <origin xyz="0.01905 -0.00107 0" rpy="0 0 0" />
         <mass value="0.00538"/>
         <inertia ixx= "0.00000006639"
@@ -312,5 +316,5 @@
     <link name="${prefix}link_paramedian_hinge">
       <visual>
-        <origin rpy="0 0 0" xyz="0 0 0"/>
+        <origin xyz="0 0 0" rpy="0 0 0" />
         <geometry>
           <box size=".02 .02 .002"/>
@@ -318,5 +322,5 @@
       </visual>
       <collision>
-        <origin rpy="0 0 0" xyz="0 0 0"/>
+        <origin xyz="0 0 0" rpy="0 0 0" />
          <geometry>
           <box size=".02 .02 .002"/>
@@ -324,5 +328,5 @@
       </collision>
       <inertial>
-        <origin rpy="0 0 0" xyz="-0.01025 0.00046 0"/>
+        <origin xyz="-0.01025 0.00046 0" rpy="0 0 0" />
         <mass value="0.00276"/>
         <inertia ixx= "0.00000004213"
@@ -341,5 +345,5 @@
     <link name="${prefix}link_median_bar_underactuated">
       <visual>
-        <origin rpy="0 0 0" xyz="0.01905 0 0"/>
+        <origin xyz="0.01905 0 0" rpy="0 0 0" />
         <geometry>
           <box size="0.0381 .0075 .002"/>
@@ -347,5 +351,5 @@
       </visual>
       <collision>
-        <origin rpy="0 0 0" xyz="0.01905 0 0"/>
+        <origin xyz="0.01905 0 0" rpy="0 0 0" />
          <geometry>
           <box size="0.0381 .0075 .002"/>
@@ -353,5 +357,5 @@
       </collision>
       <inertial>
-        <origin rpy="0 0 0" xyz="0.01905 -0.00107 0"/>
+        <origin xyz="0.01905 -0.00107 0" rpy="0 0 0" />
         <mass value="0.00538"/>
         <inertia ixx= "0.00000006639"
@@ -370,5 +374,5 @@
     <link name="${prefix}link_paradistal_hinge">
       <visual>
-        <origin rpy="0 0 0" xyz="0 0 0"/>
+        <origin xyz="0 0 0" rpy="0 0 0" />
         <geometry>
           <box size=".02 .02 .002"/>
@@ -376,5 +380,5 @@
       </visual>
       <collision>
-        <origin rpy="0 0 0" xyz="0 0 0"/>
+        <origin xyz="0 0 0" rpy="0 0 0" />
          <geometry>
           <box size=".02 0.02 .002"/>
@@ -382,5 +386,5 @@
       </collision>
       <inertial>
-        <origin rpy="0 0 0" xyz="0.00548 0 0"/>
+        <origin xyz="0.00548 0 0" rpy="0 0 0" />
         <mass value="0.00158"/>
         <inertia ixx= "0.00000001907"
@@ -403,6 +407,6 @@
       <child link="${prefix}link_proximal_actuating_hinge"/>
       <axis xyz="0 0 1"/>
-      <origin rpy="0 0 -2.0906" xyz="0 0 0.01"/>
-      <limit effort="100" lower="-3.1416" upper="3.1416" velocity="100"/>
+      <origin xyz="0 0 0.01" rpy="0 0 -2.0906" />
+      <limit effort="100" lower="${-M_PI}" upper="${M_PI}" velocity="100"/>
     </joint>
     <gazebo reference="${prefix}joint_proximal_actuating_hinge">
@@ -414,6 +418,6 @@
       <child link="${prefix}link_paraproximal_actuating_hinge"/>
       <axis xyz="0 0 1"/>
-      <origin rpy="0 0 -2.0906" xyz="0 0 -0.01"/>
-      <limit effort="100" lower="-3.1416" upper="3.1416" velocity="100"/>
+      <origin xyz="0 0 -0.01" rpy="0 0 -2.0906" />
+      <limit effort="100" lower="${-M_PI}" upper="${M_PI}" velocity="100"/>
     </joint>
     <gazebo reference="${prefix}joint_paraproximal_actuating_hinge">
@@ -425,6 +429,6 @@
       <child link="${prefix}link_proximal_actuating_bar"/>
       <axis xyz="0 0 1"/>
-      <origin rpy="0 0 1.8616" xyz="0.02858 0 0"/>
-      <limit effort="100" lower="-3.1416" upper="3.1416" velocity="100"/>
+      <origin xyz="0.02858 0 0" rpy="0 0 1.8616" />
+      <limit effort="100" lower="${-M_PI}" upper="${M_PI}" velocity="100"/>
     </joint>
     <gazebo reference="${prefix}joint_proximal_actuating_bar">
@@ -436,6 +440,6 @@
       <child link="${prefix}link_paraproximal_bar"/>
       <axis xyz="0 0 1"/>
-      <origin rpy="0 0 1.57" xyz="0.02286 0 0"/>
-      <limit effort="100" lower="-3.1416" upper="3.1416" velocity="100"/>
+      <origin xyz="0.02286 0 0" rpy="0 0 1.57" />
+      <limit effort="100" lower="${-M_PI}" upper="${M_PI}" velocity="100"/>
     </joint>
     <gazebo reference="${prefix}joint_paraproximal_bar">
@@ -447,6 +451,6 @@
       <child link="${prefix}link_median_actuating_hinge"/>
       <axis xyz="0 0 1"/>
-      <origin rpy="0 0 ${-0.37}" xyz="0 0.05715 0.01"/>
-      <limit effort="100" lower="-3.1416" upper="3.1416" velocity="100"/>
+      <origin xyz="0 0.05715 0.01" rpy="0 0 ${-0.37}" />
+      <limit effort="100" lower="${-M_PI}" upper="${M_PI}" velocity="100"/>
     </joint>
     <gazebo reference="${prefix}joint_median_actuating_hinge">
@@ -459,6 +463,6 @@
       <axis xyz="0 0 1"/>
       <!-- -0.37 is hand picked, 0.9719 is hand calculated from atan(0.02381/0.01625) -->
-      <origin rpy="0 0 0" xyz="0 0.05715 -0.01"/>
-      <limit effort="100" lower="-3.1416" upper="3.1416" velocity="100"/>
+      <origin xyz="0 0.05715 -0.01" rpy="0 0 0" />
+      <limit effort="100" lower="${-M_PI}" upper="${M_PI}" velocity="100"/>
     </joint>
     <gazebo reference="${prefix}joint_paramedian_hinge">
@@ -471,6 +475,6 @@
       <axis xyz="0 0 1"/>
       <!-- hand calc 90 deg + atan(0.01516/0.01625) -->
-      <origin rpy="0 0 ${3.1416/2 + 0.7507}" xyz="0.01625 0.01516 0"/>
-      <limit effort="100" lower="-3.1416" upper="3.1416" velocity="100"/>
+      <origin xyz="0.01625 0.01516 0" rpy="0 0 ${M_PI/2 + 0.7507}" />
+      <limit effort="100" lower="${-M_PI}" upper="${M_PI}" velocity="100"/>
     </joint>
     <gazebo reference="${prefix}joint_median_actuating_hinge_median_bar">
@@ -482,6 +486,6 @@
       <child link="${prefix}link_paradistal_hinge"/>
       <axis xyz="0 0 1"/>
-      <origin rpy="0 0 0" xyz="0 0.039 -0.01"/>
-      <limit effort="100" lower="-3.1416" upper="3.1416" velocity="100"/>
+      <origin xyz="0 0.039 -0.01" rpy="0 0 0" />
+      <limit effort="100" lower="${-M_PI}" upper="${M_PI}" velocity="100"/>
     </joint>
     <gazebo reference="${prefix}joint_paradistal_hinge">
@@ -494,6 +498,6 @@
       <axis xyz="0 0 1"/>
       <!-- hand calc 90 deg + atan(0.01227/0.00329) -->
-      <origin rpy="0 0 ${3.1416/2}" xyz="0.01227 0.00329 0"/>
-      <limit effort="100" lower="-3.1416" upper="3.1416" velocity="100"/>
+      <origin xyz="0.01227 0.00329 0" rpy="0 0 ${M_PI/2}" />
+      <limit effort="100" lower="${-M_PI}" upper="${M_PI}" velocity="100"/>
     </joint>
     <gazebo reference="${prefix}joint_paramedian_hinge_median_bar_underactuated">
@@ -502,5 +506,5 @@
     <!-- Joint 1 -->
     <joint name="${prefix}joint_1" type="revolute">
-      <origin rpy="0 0 -2.0906" xyz="0 0 0"/>
+      <origin xyz="0 0 0" rpy="0 0 -2.0906" />
       <axis xyz="0 0 1" />
       <parent link="${prefix}link_0"/>
@@ -519,5 +523,5 @@
       <dynamics damping="1" friction="0" />
       <axis xyz="0 0 1"/>
-      <origin rpy="0 0 0" xyz="0 0.05715 0"/>
+      <origin xyz="0 0.05715 0" rpy="0 0 0" />
       <!-- Limits: [0deg.,90deg.] -->
       <limit lower="0" upper="1.5708" effort="60" velocity="-1"/>
@@ -532,5 +536,5 @@
       <dynamics damping="1" friction="0" />
       <axis xyz="0 0 1"/>
-      <origin rpy="0 0 ${3.1416/2 + 0.5198}" xyz="0 0.039 0"/>
+      <origin xyz="0 0.039 0" rpy="0 0 ${M_PI/2 + 0.5198}" />
       <!-- Limits: [-38deg.,60deg.] -->
       <limit lower="-0.6632" upper="1.0471" effort="60" velocity="-1"/>
@@ -656,5 +660,5 @@
         <!-- Simple shape collision -->
         <collision>
-          <origin rpy="0 0 0" xyz="0 0 0"/>
+          <origin xyz="0 0 0" rpy="0 0 0"/>
           <geometry>
             <box size="0.1 0.1 0.1"/>
@@ -665,5 +669,5 @@
         </collision>
         <inertial>
-          <origin rpy="0 0 0" xyz="0 0 0"/>
+          <origin xyz="0 0 0" rpy="0 0 0"/>
           <mass value="1.3"/>
           <inertia ixx="0.0035" ixy="0" ixz="-0" iyy="0.0035" iyz="0" izz="0.0035"/>
@@ -682,5 +686,5 @@
       <dynamics damping="1" friction="0" />
       <axis xyz="0 1 0"/>
-      <origin rpy="0 3.1416 -1.57" xyz="-0.0455 0.0214 0.036"/>
+      <origin xyz="-0.0455 0.0214 0.036" rpy="0 ${M_PI} -1.57" />
       <!-- Limits: [-17deg.,17deg.] -->
       <limit lower="-0.2967" upper="0.2967" effort="60" velocity="-1"/>
@@ -695,5 +699,5 @@
       <dynamics damping="1" friction="0" />
       <axis xyz="0 1 0"/>
-      <origin rpy="0 3.1416 -1.57" xyz="-0.0455 0.0214 -0.036"/>
+      <origin xyz="-0.0455 0.0214 -0.036" rpy="0 ${M_PI} -1.57" />
       <!-- Limits: [-17deg.,17deg.] -->
       <limit lower="-0.2967" upper="0.2967" effort="60" velocity="-1"/>
@@ -708,5 +712,5 @@
       <dynamics damping="1" friction="0" />
       <axis xyz="0 1 0"/>
-      <origin rpy="0 0 1.57" xyz="0.0455 0.0214 0"/>
+      <origin xyz="0.0455 0.0214 0" rpy="0 0 1.57" />
       <limit lower="0" upper="0" effort="60" velocity="-1"/>
     </joint>
@@ -716,5 +720,5 @@
       <parent link="${prefix}palm"/>
       <child link="grasping_frame"/>
-      <origin xyz="0 0.1 0.01" rpy="0 -1.5708 3.14159"/>
+      <origin xyz="0 0.1 0.01" rpy="0 -1.5708 3.14159"  />
     </joint>
     <gazebo reference="${prefix}palm_finger_middle_joint">

Commit message: update

File: robotiq/robotiq_s_model_visualization/cfg/robotiq_hand_macro.urdf.xacro (robot description, xacro)
@@ -11,4 +11,12 @@
     <!-- Gripper frame -->
   <xacro:property name="grasp_frame_radius" value="0.001" />
+    <!-- Defining the colors used in this robot -->
+  <material name="green"><color rgba="0 1 0 1"/></material>
+  <material name="dark_grey_iq"><color rgba="0.2 0.2 0.2 1.0" /></material>
+  <material name="light_grey_iq"><color rgba="0.4 0.4 0.4 1.0" /></material>
+  <material name="red_iq"><color rgba="0.8 0.0 0.0 1.0" /></material>
+  <material name="white_iq"><color rgba="0.9 0.9 0.9 1.0" /></material>
+  <material name="yellow_iq"><color rgba="0.8 0.8 0.0 1.0" /></material>
+  <material name="black_iq"><color rgba="0.15 0.15 0.15 1.0" /></material>
   <xacro:macro name="robotiq_finger" params="prefix">
     <!-- Link list -->
@@ -20,7 +28,5 @@
           <mesh filename="package://robotiq_s_model_visualization/meshes/s-model_articulated/visual/link_0.STL" />
         </geometry>
-        <material name="green">
-          <color rgba="0 1 0 1"/>
-        </material>
+        <material name="green" />
       </visual>
       <collision>
@@ -29,7 +35,5 @@
           <mesh filename="package://robotiq_s_model_visualization/meshes/s-model_articulated/collision/link_0.STL" />
         </geometry>
-        <material name="yellow">
-          <color rgba="0 1 1 1"/>
-        </material>
+        <material name="yellow_iq" />
       </collision>
       <inertial>
@@ -57,7 +61,5 @@
           <mesh filename="package://robotiq_s_model_visualization/meshes/s-model_articulated/collision/link_1.STL"/>
         </geometry>
-        <material name="yellow">
-          <color rgba="0 1 1 1"/>
-        </material>
+        <material name="yellow_iq" />
       </collision>
       <inertial>
@@ -90,5 +92,5 @@
             <mesh filename="package://robotiq_s_model_visualization/meshes/s-model_articulated/collision/link_2.STL"/>
           </geometry>
-        <material name="yellow"/>
+        <material name="yellow_iq"/>
       </collision>
       <inertial>
@@ -121,5 +123,5 @@
           <mesh filename="package://robotiq_s_model_visualization/meshes/s-model_articulated/collision/link_3.STL"/>
         </geometry>
-        <material name="yellow"/>
+        <material name="yellow_iq"/>
       </collision>
       <inertial>
@@ -654,7 +656,5 @@
             <mesh filename="package://robotiq_s_model_visualization/meshes/s-model_articulated/visual/palm.STL" />
           </geometry>
-          <material name="green">
-            <color rgba="0 1 0 1"/>
-          </material>
+          <material name="green" />
         </visual>
         <!-- Simple shape collision -->
@@ -664,7 +664,5 @@
             <box size="0.1 0.1 0.1"/>
           </geometry>
-          <material name="yellow">
-            <color rgba="0 1 1 1"/>
-          </material>
+          <material name="yellow_iq" />
         </collision>
         <inertial>

Commit message: update

File: robotiq/robotiq_s_model_visualization/cfg/robotiq_hand_macro.urdf.xacro (robot description, xacro)
@@ -28,5 +28,5 @@
           <mesh filename="package://robotiq_s_model_visualization/meshes/s-model_articulated/visual/link_0.STL" />
         </geometry>
-        <material name="green" />
+        <material name="black_iq" />
       </visual>
       <collision>
@@ -35,5 +35,5 @@
           <mesh filename="package://robotiq_s_model_visualization/meshes/s-model_articulated/collision/link_0.STL" />
         </geometry>
-        <material name="yellow_iq" />
+        <material name="black_iq" />
       </collision>
       <inertial>
@@ -54,5 +54,5 @@
           <mesh filename="package://robotiq_s_model_visualization/meshes/s-model_articulated/visual/link_1.STL" />
         </geometry>
-        <material name="green"/>
+        <material name="black_iq"/>
       </visual>
       <collision>
@@ -61,5 +61,5 @@
           <mesh filename="package://robotiq_s_model_visualization/meshes/s-model_articulated/collision/link_1.STL"/>
         </geometry>
-        <material name="yellow_iq" />
+        <material name="black_iq" />
       </collision>
       <inertial>
@@ -85,5 +85,5 @@
           <mesh filename="package://robotiq_s_model_visualization/meshes/s-model_articulated/visual/link_2.STL" />
         </geometry>
-        <material name="green"/>
+        <material name="black_iq"/>
       </visual>
       <collision>
@@ -92,5 +92,5 @@
             <mesh filename="package://robotiq_s_model_visualization/meshes/s-model_articulated/collision/link_2.STL"/>
           </geometry>
-        <material name="yellow_iq"/>
+        <material name="black_iq"/>
       </collision>
       <inertial>
@@ -116,5 +116,5 @@
           <mesh filename="package://robotiq_s_model_visualization/meshes/s-model_articulated/visual/link_3.STL" />
         </geometry>
-        <material name="green"/>
+        <material name="white_iq"/>
       </visual>
       <collision>
@@ -123,5 +123,5 @@
           <mesh filename="package://robotiq_s_model_visualization/meshes/s-model_articulated/collision/link_3.STL"/>
         </geometry>
-        <material name="yellow_iq"/>
+        <material name="black_iq"/>
       </collision>
       <inertial>
@@ -656,5 +656,5 @@
             <mesh filename="package://robotiq_s_model_visualization/meshes/s-model_articulated/visual/palm.STL" />
           </geometry>
-          <material name="green" />
+          <material name="black_iq" />
         </visual>
         <!-- Simple shape collision -->
@@ -664,5 +664,5 @@
             <box size="0.1 0.1 0.1"/>
           </geometry>
-          <material name="yellow_iq" />
+          <material name="black_iq" />
         </collision>
         <inertial>
