Commit message: update robotiq_hand_macro.urdf.xacro

File: robotiq_3f_gripper_visualization/cfg/robotiq_hand_macro.urdf.xacro (robot description, xacro)
@@ -16,7 +16,5 @@
           <mesh filename="package://robotiq_3f_gripper_visualization/meshes/robotiq-3f-gripper_articulated/visual/link_0.STL" />
         </geometry>
-        <material name="green">
-          <color rgba="0 1 0 1"/>
-        </material>
+      <material name="black"/>
       </visual>
       <collision>
@@ -46,5 +44,5 @@
           <mesh filename="package://robotiq_3f_gripper_visualization/meshes/robotiq-3f-gripper_articulated/visual/link_1.STL" />
         </geometry>
-        <material name="green"/>
+        <material name="black"/>
       </visual>
       <collision>
@@ -79,5 +77,5 @@
           <mesh filename="package://robotiq_3f_gripper_visualization/meshes/robotiq-3f-gripper_articulated/visual/link_2.STL" />
         </geometry>
-        <material name="green"/>
+        <material name="black"/>
       </visual>
       <collision>
@@ -110,5 +108,5 @@
           <mesh filename="package://robotiq_3f_gripper_visualization/meshes/robotiq-3f-gripper_articulated/visual/link_3.STL" />
         </geometry>
-        <material name="green"/>
+        <material name="white"/>
       </visual>
       <collision>
@@ -141,4 +139,5 @@
           <box size="0.02858 .0075 .002"/>
         </geometry>
+ <material name="black"/>
       </visual>
       <collision>
@@ -170,4 +169,5 @@
           <box size="0.02286 .0075 .002"/>
         </geometry>
+ <material name="black"/>
       </visual>
       <collision>
@@ -200,4 +200,5 @@
           <box size="0.05398 .0075 .002"/>
         </geometry>
+ <material name="black"/>
       </visual>
       <collision>
@@ -229,4 +230,5 @@
           <box size="0.05770 .0075 .002"/>
         </geometry>
+ <material name="black"/>
       </visual>
       <collision>
@@ -258,4 +260,5 @@
           <box size=".02 .02 .002"/>
         </geometry>
+ <material name="black"/>
       </visual>
       <collision>
@@ -287,4 +290,5 @@
           <box size="0.0381 .0075 .002"/>
         </geometry>
+ <material name="black"/>
       </visual>
       <collision>
@@ -316,4 +320,5 @@
           <box size=".02 .02 .002"/>
         </geometry>
+ <material name="black"/>
       </visual>
       <collision>
@@ -345,4 +350,5 @@
           <box size="0.0381 .0075 .002"/>
         </geometry>
+ <material name="black"/>
       </visual>
       <collision>
@@ -374,4 +380,5 @@
           <box size=".02 .02 .002"/>
         </geometry>
+ <material name="black"/>
       </visual>
       <collision>
@@ -650,7 +657,5 @@
             <mesh filename="package://robotiq_3f_gripper_visualization/meshes/robotiq-3f-gripper_articulated/visual/palm.STL" />
           </geometry>
-          <material name="green">
-            <color rgba="0 1 0 1"/>
-          </material>
+        <material name="black"/>
         </visual>
         <!-- Simple shape collision -->
