Commit message: update gazebo

File: robotiq_3f_gripper_visualization/cfg/robotiq-3f-gripper_articulated_macro.xacro (robot description, xacro)
@@ -1,2 +1,3 @@
+<?xml version="1.0" ?>
 <!--
 robotiq-3f-gripper_articulated_macro(prefix)
@@ -6,14 +7,14 @@
 -->
 <robot xmlns:xacro="http://ros.org/wiki/xacro">
-        <xacro:include filename="$(find robotiq_3f_gripper_visualization)/cfg/robotiq-3f-gripper_finger_articulated_macro.xacro" />
-        <xacro:macro name="robotiq-3f-gripper_articulated" params="prefix">
-        <xacro:robotiq-3f-gripper_finger_articulated prefix="${prefix}finger_1_"/>
-        <xacro:robotiq-3f-gripper_finger_articulated prefix="${prefix}finger_2_"/>
-        <xacro:robotiq-3f-gripper_finger_articulated prefix="${prefix}finger_middle_"/>
+    <xacro:include filename="$(find robotiq_3f_gripper_visualization)/cfg/robotiq-3f-gripper_finger_articulated_macro.xacro" />
+    <xacro:macro name="robotiq-3f-gripper_articulated" params="prefix">
+    <xacro:robotiq-3f-gripper_finger_articulated prefix="${prefix}finger_1_"/>
+    <xacro:robotiq-3f-gripper_finger_articulated prefix="${prefix}finger_2_"/>
+    <xacro:robotiq-3f-gripper_finger_articulated prefix="${prefix}finger_middle_"/>
 		<!-- link list -->
 		<link name="${prefix}palm">
 			<visual>
 				<geometry>
-                                        <mesh filename="package://robotiq_3f_gripper_visualization/meshes/robotiq-3f-gripper_articulated/visual/palm.STL" />
+                	<mesh filename="package://robotiq_3f_gripper_visualization/meshes/robotiq-3f-gripper_articulated/visual/palm.STL" />
 				</geometry>
 				<material name="gray">
@@ -23,5 +24,5 @@
 			<collision>
 				<geometry>
-                                        <mesh filename="package://robotiq_3f_gripper_visualization/meshes/robotiq-3f-gripper_articulated/collision/palm.STL" />
+                    <mesh filename="package://robotiq_3f_gripper_visualization/meshes/robotiq-3f-gripper_articulated/collision/palm.STL" />
 				</geometry>
 				<material name="yellow">
@@ -30,5 +31,11 @@
 			</collision>
 		</link>
+		<gazebo reference="${prefix}palm">
+            <material>Gazebo/Black</material>
+       	</gazebo>
 		<link name="${prefix}tool0"/>
+        <gazebo reference="${prefix}tool0">
+            <material>Gazebo/Blue</material>
+        </gazebo>
         <inertial>
             <origin xyz="0 0 0" rpy="0 0 0"/>
@@ -45,4 +52,14 @@
 			<limit lower="-0.1784" upper="0.192" effort="100" velocity="100"/>
 		</joint>
+        <transmission name="${prefix}palm_finger_1_joint_trans">
+            <type>transmission_interface/SimpleTransmission</type>
+            <joint name="${prefix}palm_finger_1_joint" >
+                <hardwareInterface>hardware_interface/VelocityJointInterface</hardwareInterface>
+            </joint>
+            <actuator name="${prefix}palm_finger_1_joint_motor">
+                <hardwareInterface>hardware_interface/VelocityJointInterface</hardwareInterface>
+                <mechanicalReduction>1</mechanicalReduction>
+            </actuator>
+        </transmission>
 		<joint name="${prefix}palm_finger_2_joint" type="revolute">
 			<parent link="${prefix}palm"/>
@@ -52,4 +69,14 @@
 			<limit lower="-0.192" upper="0.1784" effort="100" velocity="100"/>
 		</joint>
+        <transmission name="${prefix}palm_finger_2_joint_trans">
+            <type>transmission_interface/SimpleTransmission</type>
+            <joint name="${prefix}palm_finger_2_joint" >
+                <hardwareInterface>hardware_interface/VelocityJointInterface</hardwareInterface>
+            </joint>
+            <actuator name="${prefix}palm_finger_2_joint_motor">
+                <hardwareInterface>hardware_interface/VelocityJointInterface</hardwareInterface>
+                <mechanicalReduction>1</mechanicalReduction>
+            </actuator>
+        </transmission>
 		<joint name="${prefix}palm_finger_middle_joint" type="fixed">
 			<parent link="${prefix}palm"/>
@@ -58,4 +85,14 @@
 			<origin xyz="0.0455 0.0214 0" rpy="0 0 1.57"/>
 		</joint>
+        <transmission name="${prefix}palm_finger_middle_joint_trans">
+            <type>transmission_interface/SimpleTransmission</type>
+            <joint name="${prefix}palm_finger_middle_joint" >
+                <hardwareInterface>hardware_interface/VelocityJointInterface</hardwareInterface>
+            </joint>
+            <actuator name="${prefix}palm_finger_middle_joint_motor">
+                <hardwareInterface>hardware_interface/VelocityJointInterface</hardwareInterface>
+                <mechanicalReduction>1</mechanicalReduction>
+            </actuator>
+        </transmission>
 		<joint name="${prefix}palm_tool0" type="fixed">
 			<parent link="${prefix}palm"/>
