Commit message: add robotiq_hand

File: robotiq_3f_gripper_visualization/cfg/robotiq-3f-gripper_mesh_macro.xacro (robot description, xacro)
@@ -1,2 +1,3 @@
+<?xml version="1.0" ?>
 <robot xmlns:xacro="http://ros.org/wiki/xacro">
         <xacro:macro name="robotiq-3f-gripper_mesh" params="prefix">

File: robotiq_3f_gripper_visualization/cfg/ur5_robotiq-3f-gripper_finger_articulated_macro.xacro (robot description, xacro)
@@ -1,3 +1,3 @@
-<?xml version="1.0" ?>
+<?xml version='1.0' encoding='utf-8'?>
 <!--
 robotiq-3f-gripper_finder_articulated_macro(prefix)
@@ -6,14 +6,21 @@
 finger(i.e. finger_1, etc...).
 -->
-<robot xmlns:xacro="http://ros.org/wiki/xacro">
-        <xacro:macro name="robotiq-3f-gripper_finger_articulated" params="prefix">
-		<!-- link list -->
-		<link name="${prefix}link_0">
-			<visual>
-				<origin xyz="0.020 0 0" rpy="0 0 0"/>
-				<geometry>
-                                        <mesh filename="package://robotiq_3f_gripper_visualization/meshes/robotiq-3f-gripper_articulated/visual/link_0.STL" />
-				</geometry>
-				<material name="gray">
+<robot xmlns:xacro="http://ros.org/wiki/xacro" name="robotiq_hand">
+  <xacro:macro name="robotiq_hand" params="prefix connected_to:='' rpy:='0 0 0' xyz:='0 0 0'">
+    <xacro:unless value="${connected_to == ''}">
+      <joint name="${prefix}ur5_robotiq_joint" type="fixed">
+        <parent link="${connected_to}"/>
+        <child link="${prefix}link_0"/>
+        <origin xyz="${xyz}" rpy="${rpy}"/>
+      </joint>
+    </xacro:unless>
+	<!-- link list -->
+	<link name="${prefix}link_0">
+	<visual>
+		<origin xyz="0.020 0 0" rpy="0 0 0"/>
+		<geometry>
+                <mesh filename="package://robotiq_3f_gripper_visualization/meshes/robotiq-3f-gripper_articulated/visual/link_0.STL" />
+		</geometry>
+		<material name="gray">
 					<color rgba="0.2 0.2 0.2 1"/>
 				</material>

File: robotiq_3f_gripper_visualization/urdf/robotiq-hand.xacro (robot description, xacro)
@@ -1,3 +1,3 @@
-<?xml version="1.0" ?>
+<?xml version="1.0" encoding="utf-8"?>
 <!--
 robotiq-3f-gripper_finder_articulated_macro(prefix)
@@ -7,5 +7,5 @@
 -->
 <robot xmlns:xacro="http://ros.org/wiki/xacro">
-        <xacro:macro name="robotiq-3f-gripper_finger_articulated" params="prefix">
+        <xacro:macro name="robotiq_hand" params="prefix">
 		<!-- link list -->
 		<link name="${prefix}link_0">

File: robotiq_3f_gripper_visualization/urdf/robotiq_articulated_macro.xacro (robot description, xacro)
@@ -1,3 +1,3 @@
-<?xml version="1.0" ?>
+<?xml version="1.0" encoding="utf-8"?>
 <!--
 robotiq-3f-gripper_articulated_macro(prefix)
@@ -7,9 +7,16 @@
 -->
 <robot xmlns:xacro="http://ros.org/wiki/xacro">
-    <xacro:include filename="$(find robotiq_3f_gripper_visualization)/cfg/robotiq-3f-gripper_finger_articulated_macro.xacro" />
-    <xacro:macro name="robotiq-3f-gripper_articulated" params="prefix">
-    <xacro:robotiq-3f-gripper_finger_articulated prefix="${prefix}finger_1_"/>
-    <xacro:robotiq-3f-gripper_finger_articulated prefix="${prefix}finger_2_"/>
-    <xacro:robotiq-3f-gripper_finger_articulated prefix="${prefix}finger_middle_"/>
+    <xacro:include filename="$(find robotiq_3f_gripper_visualization)/urdf/robotiq-hand.xacro" />
+    <xacro:macro name="robotiq_articulated_macro" params="prefix connected_to:='' rpy:='0 0 0' xyz:='0 0 0'">
+    <xacro:robotiq_hand prefix="${prefix}finger_1_"/>
+    <xacro:robotiq_hand prefix="${prefix}finger_2_"/>
+    <xacro:robotiq_hand prefix="${prefix}finger_middle_"/>
+    <xacro:unless value="${connected_to == ''}">
+      <joint name="${prefix}ur5_robotiq_joint" type="fixed">
+        <parent link="${connected_to}"/>
+        <child link="${prefix}palm"/>
+        <origin xyz="${xyz}" rpy="${rpy}"/>
+      </joint>
+    </xacro:unless>
 		<!-- link list -->
 		<link name="${prefix}palm">
@@ -40,5 +47,5 @@
         <inertial>
             <origin xyz="0 0 0" rpy="0 0 0"/>
-            <mass value="1.3"/>
+            <mass value="0.5"/>
             <inertia ixx="0.006012" ixy="0.000079" ixz="-0.00024" iyy="0.012892" iyz="0" izz="0.002435" />
         </inertial>
@@ -85,5 +92,5 @@
 			<origin xyz="0.0455 0.0214 0" rpy="0 0 1.57"/>
 		</joint>
-        <transmission name="${prefix}palm_finger_middle_joint_trans">
+        <!--transmission name="${prefix}palm_finger_middle_joint_trans">
             <type>transmission_interface/SimpleTransmission</type>
             <joint name="${prefix}palm_finger_middle_joint" >
@@ -94,5 +101,5 @@
                 <mechanicalReduction>1</mechanicalReduction>
             </actuator>
-        </transmission>
+        </transmission-->
 		<joint name="${prefix}palm_tool0" type="fixed">
 			<parent link="${prefix}palm"/>
